File: hw/ver1/ws2812.kicad_sch (KiCad schematic)
At the start: 2 parts

Commit message: Nearly have all the LEDs wired up. Improve the christmas cheer.
Parts:
- renumbered C30 to C18, D13 to D1

Commit message: Hardware version 1 complete and ordered.
Parts:
- D11: renamed from D1; JLCPCB Rotation Offset (none) -> -180
- renumbered C18 to C28
